File: 1802-Mini-I2C.kicad_pcb (KiCad board)
At the start: 2 copper layers, 89 x 37 mm, 24 parts, among them J1 PORT1, J2 Qwiic, J3 PORT2, J4 Qwiic, J5 I2C_5V, J6 I2C_5V, Q1 2N3904, Q2 TN0702, Q3 TN0702, Q4 2N3904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

Commit message: Update design and add BOM
Parts:
- moved JP1 5.30 mm to (151.8, 85.0), turned to 90 degrees
- moved J5 2.06 mm to (135.4, 113.0)
- moved J6 2.06 mm to (166.9, 113.0)
- moved JP2 1.36 mm to (133.1, 91.6)
- moved JP3 1.36 mm to (133.1, 103.0)
- moved Q1 1.36 mm to (180.3, 92.5)
- moved Q2 1.36 mm to (154.0, 91.6)
- moved Q3 1.36 mm to (154.0, 102.6)
- moved Q4 1.36 mm to (180.3, 104.0)
- moved R1 1.36 mm to (171.8, 95.2)
- moved R2 1.36 mm to (171.8, 90.3)
- moved R3 1.36 mm to (147.1, 90.3)
- moved R4 1.36 mm to (147.1, 95.2)
- moved R5 1.36 mm to (171.8, 106.6)
- moved R6 1.36 mm to (171.8, 101.8)
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Connections:
- J2 pad 1: SCL_LO -> GND
- J2 pad 2: SDA_LO -> +3.3V
- J2 pad 3: +3.3V -> SDA_LO
- J2 pad 4: GND -> SCL_LO
- J4 pad 1: SCL_LO -> GND
- J4 pad 2: SDA_LO -> +3.3V
- J4 pad 3: +3.3V -> SDA_LO
- J4 pad 4: GND -> SCL_LO
- J5 pad 1: SCL_HI -> GND
- J5 pad 2: SDA_HI -> +5V
- J5 pad 3: +5V -> SDA_HI
- J5 pad 4: GND -> SCL_HI
- J6 pad 1: SCL_HI -> GND
- J6 pad 2: SDA_HI -> +5V
- J6 pad 3: +5V -> SDA_HI
- J6 pad 4: GND -> SCL_HI
Routing:
- net GND: track 38.9 -> 0.00 mm, vias 1 -> 0
- net SCL_LO: track 73.9 -> 53.2 mm
- net +5V: track 134.8 -> 124.0 mm
- net +3.3V: track 78.8 -> 87.3 mm
- net /BUS6: track 109.5 -> 105.3 mm
- net /BUS5: track 82.5 -> 86.1 mm
- net SDA_HI: track 82.1 -> 78.7 mm, vias 0 -> 1
- net SCL_HI: track 63.7 -> 67.1 mm
- net SR: track 82.0 -> 85.1 mm
- net /BUS4: track 82.0 -> 85.1 mm
- net Q: track 82.1 -> 85.1 mm
- net /BUS3: track 82.5 -> 85.1 mm
- net SDA_LO: track 39.6 -> 37.6 mm
- net /BUS7: track 82.8 -> 84.5 mm
- net /BUS2: track 84.2 -> 83.1 mm
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Other:
- board text added: "1"
- board text added: "1802/MINI"
- board text added: "3"
- board text added: "3.3V PU EN"
- board text added: "4"
- board text added: "5V"
- board text added: "5V PU EN"
- board text added: "EF SEL"
- board text added: "GND"
- board text added: "I2C ADAPTER"
- board text added: "JLCJLCJLCJLC"
- board text added: "JLCPCB ORDER #"
- board text added: "Qwiic"
- board text added: "SCL"
- board text added: "SDA"
- board text added: "rev A"
