File: 1802-Mini-I2C.kicad_sch (KiCad schematic)
At the start: 24 parts, among them J1 PORT1, J2 Qwiic, J3 PORT2, J4 Qwiic, J5 I2C_5V, J6 I2C_5V, Q1 2N3904, Q2 TN0702, Q3 TN0702, Q4 2N3904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

Commit message: Update design and add BOM
Connections:
- net +3.3V: now also J2.2, J4.2; no longer J2.3, J4.3
- net +5V: now also J5.2 (Pin_2), J6.2 (Pin_2); no longer J5.3 (Pin_3), J6.3 (Pin_3)
- net GND: now also J2.1, J4.1, J5.1 (Pin_1), J6.1 (Pin_1); no longer J2.4, J4.4, J5.4 (Pin_4), J6.4 (Pin_4)
- net SCL_HI: now also J5.4 (Pin_4), J6.4 (Pin_4); no longer J5.1 (Pin_1), J6.1 (Pin_1)
- net SCL_LO: now also J2.4, J4.4; no longer J2.1, J4.1
- net SDA_HI: now also J5.3 (Pin_3), J6.3 (Pin_3); no longer J5.2 (Pin_2), J6.2 (Pin_2)
- net SDA_LO: now also J2.3, J4.3; no longer J2.2, J4.2
